Commit message: improve urdf

File: double_pendulum.urdf (robot description, URDF)
Before this commit: robot double_pendulum, 3 links, 2 joints
Links:
- added link joint1_sphere; visual sphere radius=0.05
- added link joint2_sphere; visual sphere radius=0.05
- link base_link: mass 1.0 -> None; geometry visual box size=0.2 0.2 0.2
- link link1: mass 1.0 -> None; geometry visual cylinder length=1.0 radius=0.05
- link link2: mass 1.0 -> None; geometry visual cylinder length=1.0 radius=0.05
Joints:
- added joint joint1_link: type fixed, parent joint1_sphere, child link1, origin xyz=0 0 0 rpy=0 0 0
- added joint joint2_link: type fixed, parent joint2_sphere, child link2, origin xyz=0 0 0 rpy=0 0 0
- joint joint1: child link1 -> joint1_sphere; limit lower=-3.14 upper=3.14 effort=10 velocity=5 -> lower=-3.14 upper=3.14 effort=10 velocity=10; origin xyz=0 0 0 -> xyz=0 0 0.1 rpy=0 0 0
- joint joint2: child link2 -> joint2_sphere; limit lower=-3.14 upper=3.14 effort=10 velocity=5 -> lower=-3.14 upper=3.14 effort=10 velocity=10; origin xyz=0 0 -1.0 -> xyz=0 0 -1.0 rpy=0 0 0
